Commit message: Add support for the Gazebo simulator

File: ur_description/urdf/ur.ros2_control.xacro (robot description, xacro)
@@ -5,13 +5,16 @@
     script_filename output_recipe_filename
     input_recipe_filename tf_prefix
-    hash_kinematics robot_ip">
+    hash_kinematics robot_ip controllers_file">
     <ros2_control name="${name}" type="system">
       <hardware>
-        <xacro:if value="${use_fake_hardware}">
+        <xacro:if value="${use_fake_hardware == 'gazebo'}">
+          <plugin>gazebo_ros2_control/GazeboSystem</plugin>
+        </xacro:if>
+        <xacro:if value="${use_fake_hardware == True}">
           <plugin>fake_components/GenericSystem</plugin>
           <param name="fake_sensor_commands">${fake_sensor_commands}</param>
           <param name="state_following_offset">0.0</param>
         </xacro:if>
-        <xacro:unless value="${use_fake_hardware}">
+        <xacro:if value="${use_fake_hardware == False}">
           <plugin>ur_robot_driver/URPositionHardwareInterface</plugin>
           <param name="robot_ip">${robot_ip}</param>
@@ -36,5 +39,5 @@
           <param name="tool_device_name">/tmp/ttyUR</param>
           <param name="tool_tcp_port">54321</param>
-        </xacro:unless>
+        </xacro:if>
       </hardware>
       <joint name="${prefix}shoulder_pan_joint">
@@ -225,4 +228,11 @@
       </joint>
     </ros2_control>
+    <gazebo>
+      <plugin filename="libgazebo_ros2_control.so" name="gazebo_ros2_control">
+        <robot_param>robot_description</robot_param>
+        <robot_param_node>robot_state_publisher</robot_param_node>
+        <parameters>$(arg controllers_file)</parameters>
+      </plugin>
+    </gazebo>
   </xacro:macro>
 </robot>

File: ur_description/urdf/ur.urdf.xacro (robot description, xacro)
@@ -18,4 +18,5 @@
    <xacro:arg name="use_fake_hardware" default="false" />
    <xacro:arg name="fake_sensor_commands" default="false" />
+   <xacro:arg name="controllers_file" default="" />
    <!-- arm -->
    <xacro:ur_robot
@@ -30,4 +31,5 @@
      safety_k_position="$(arg safety_k_position)"
      use_fake_hardware="$(arg use_fake_hardware)"
-     fake_sensor_commands="$(arg fake_sensor_commands)" />
+     fake_sensor_commands="$(arg fake_sensor_commands)"
+     controllers_file="$(arg controllers_file)" />
 </robot>

File: ur_description/urdf/ur_macro.xacro (robot description, xacro)
@@ -55,5 +55,6 @@
     safety_k_position:=20
     use_fake_hardware:=false
-    fake_sensor_commands:=false"
+    fake_sensor_commands:=false
+    controllers_file"
   >
     <!-- Load configuration data from the provided .yaml files -->
@@ -80,9 +81,13 @@
       tf_prefix=""
       hash_kinematics="${kinematics_hash}"
-      robot_ip="$(arg robot_ip)" />
+      robot_ip="$(arg robot_ip)"
+      controllers_file="$(arg controllers_file)" />
     <!-- Add URDF transmission elements (for ros_control) -->
     <!--<xacro:ur_arm_transmission prefix="${prefix}" hw_interface="${transmission_hw_interface}" />-->
     <!-- Placeholder for ros2_control transmission which don't yet exist -->
     <!-- links -  main serial chain -->
+    <xacro:if value="${use_fake_hardware == 'gazebo'}">
+      <link name="world"/>
+    </xacro:if>
     <link name="${prefix}base_link"/>
     <link name="${prefix}base_link_inertia">
@@ -227,4 +232,11 @@
     </link>
     <!-- joints - main serial chain -->
+    <xacro:if value="${use_fake_hardware == 'gazebo'}">
+      <joint name="world_to_base" type="fixed">
+        <origin rpy="0 0 0" xyz="0 0 1"/>
+        <parent link="world"/>
+        <child link="${prefix}base_link"/>
+      </joint>
+    </xacro:if>
     <joint name="${prefix}base_link-base_link_inertia" type="fixed">
       <parent link="${prefix}base_link" />
