Commit message: Remove world link

File: ur_description/urdf/ur_macro.xacro (robot description, xacro)
@@ -87,7 +87,4 @@
     <!-- Placeholder for ros2_control transmission which don't yet exist -->
     <!-- links -  main serial chain -->
-    <xacro:if value="${use_fake_hardware == 'gazebo'}">
-      <link name="world"/>
-    </xacro:if>
     <link name="${prefix}base_link"/>
     <link name="${prefix}base_link_inertia">
@@ -232,11 +229,4 @@
     </link>
     <!-- joints - main serial chain -->
-    <xacro:if value="${use_fake_hardware == 'gazebo'}">
-      <joint name="world_to_base" type="fixed">
-        <origin rpy="0 0 0" xyz="0 0 1"/>
-        <parent link="world"/>
-        <child link="${prefix}base_link"/>
-      </joint>
-    </xacro:if>
     <joint name="${prefix}base_link-base_link_inertia" type="fixed">
       <parent link="${prefix}base_link" />
